File: frontpanel.kicad_pcb (KiCad board)
At the start: 2 copper layers, 20 x 20 mm, 1 part

Commit message: modified adapter
Other:
- board size 20 x 20 mm -> 24 x 24 mm

Commit message: Doku for Fix
Parts:
- added REF**: TQFP-100_14x14mm_P0.5mm, Package_QFP:TQFP-100_14x14mm_P0.5mm, B.Cu at (155.0, 100.0)
